File: hardware/mppt_power_path/mppt_power_path.kicad_sch (KiCad schematic)
At the start: 79 parts, among them IC101 SN74HCS367PWR, IC102 SN74LVC1G04DBVR, IC103 SN74LVC2G32DCUR, IC104 SN74LVC08APWR, IC105 INA229AIDGSR, IC106 INA229AIDGSR, J101 CT3151, J102 CT3151, J103 CT3151, J104 CT3151, J105 CT3151, J106 CT3151, J107 CT3151, J108 CT3151, J110 Conn_01x16, Q101 Q_NMOS_GDS, Q102 Q_NMOS_GDS, Q103 Q_NMOS_GDS, Q104 BSS127S, Q109 Q_NMOS_GDS, Q110 BSS127S, U101 TPSI3050, U104 TPSI3050

Commit message: revise sch and bom for power path, prelim layout, prelim documentation structure
Parts:
- removed Q101, Q102, Q103, Q109: Q_NMOS_GDS, Package_TO_SOT_SMD:SOT-223-3_TabPin2, symbol Device:Q_NMOS_GDS
- removed R104, R127: 10k, Resistor_SMD:R_2512_6332Metric_Pad1.40x3.35mm_HandSolder, symbol Device:R_Small
- removed R116, R121: 3.2m, Resistor_SMD:R_2512_6332Metric_Pad1.40x3.35mm_HandSolder, symbol Device:R
- removed R117: 150k, symbol Device:R_Small
- added Q2, Q3, Q4, Q5: Q_NMOS_SGD, Package_SO:PowerPAK_SO-8_Single, symbol Device:Q_NMOS_SGD
- added R1: 87.5k, Resistor_SMD:R_0805_2012Metric_Pad1.20x1.40mm_HandSolder, symbol Device:R_Small
- added R10, R22: 10k, Resistor_SMD:R_2512_6332Metric_Pad1.40x3.35mm_HandSolder, symbol Device:R
- added R26, R5: 4m, Resistor_SMD:R_Shunt_Vishay_WSKW0612, symbol Device:R_Shunt
- C1: renamed from C112; footprint (none) -> Capacitor_SMD:C_0805_2012Metric_Pad1.18x1.45mm_HandSolder; Manufacturer (none) -> Samsung Microelectronics; Notes (none) -> 3.3V* guaranteed to fail on hard short from + to - rail
- C10: renamed from C105; footprint Resistor_SMD:R_0402_1005Metric -> Capacitor_SMD:C_0805_2012Metric_Pad1.18x1.45mm_HandSolder; Cost 0.0068 -> (none); Distributor LCSC -> (none); LCSC Part # C307454 -> (none); Manufacturer Samsung Electromechanics -> Samsung Microelectronics; Notes Sized according to TPSI305x calculator spreadsheet (150nC, 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 -> 10V; P/N CL05X105KA5NQNC -> (none)
- C11: renamed from C106; footprint Resistor_SMD:R_0402_1005Metric -> Capacitor_SMD:C_0805_2012Metric_Pad1.18x1.45mm_HandSolder; Cost 0.0068 -> (none); Distributor LCSC -> (none); LCSC Part # C307454 -> (none); Manufacturer Samsung Electromechanics -> Samsung Microelectronics; Notes Sized according to TPSI305x calculator spreadsheet (150nC, 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 -> 10V; P/N CL05X105KA5NQNC -> (none)
- C12: renamed from C113; footprint (none) -> Capacitor_SMD:C_0805_2012Metric_Pad1.18x1.45mm_HandSolder; Manufacturer (none) -> Samsung Microelectronics; Notes (none) -> 3.3V
- C13: renamed from C108; footprint (none) -> Capacitor_SMD:C_0805_2012Metric_Pad1.18x1.45mm_HandSolder; Manufacturer (none) -> Samsung Microelectronics; Notes (none) -> 3.3V
- C14: renamed from C111; footprint (none) -> Capacitor_SMD:C_0805_2012Metric_Pad1.18x1.45mm_HandSolder; Manufacturer (none) -> Samsung Microelectronics; Notes (none) -> 3.3V* guaranteed to fail on hard short from + to - rail
- C15: renamed from C109; footprint (none) -> Capacitor_SMD:C_0805_2012Metric_Pad1.18x1.45mm_HandSolder; Manufacturer (none) -> Samsung Microelectronics; Notes (none) -> 3.3V
- C2: renamed from C114; footprint (none) -> Capacitor_SMD:C_0805_2012Metric_Pad1.18x1.45mm_HandSolder; Manufacturer (none) -> Samsung Microelectronics; Notes (none) -> 3.3V
- C3: renamed from C115; footprint Resistor_SMD:R_0402_1005Metric -> Capacitor_SMD:C_0805_2012Metric_Pad1.18x1.45mm_HandSolder; Cost 0.0068 -> (none); Distributor LCSC -> (none); LCSC Part # C307454 -> (none); Manufacturer Samsung Electromechanics -> Samsung Microelectronics; Notes Sized according to TPSI305x calculator spreadsheet (150nC, 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 -> 10V; P/N CL05X105KA5NQNC -> (none)
- C4: renamed from C116; footprint Resistor_SMD:R_0402_1005Metric -> Capacitor_SMD:C_0805_2012Metric_Pad1.18x1.45mm_HandSolder; Cost 0.0068 -> (none); Distributor LCSC -> (none); LCSC Part # C307454 -> (none); Manufacturer Samsung Electromechanics -> Samsung Microelectronics; Notes Sized according to TPSI305x calculator spreadsheet (150nC, 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 -> 10V; P/N CL05X105KA5NQNC -> (none)
- C5: renamed from C101; footprint Resistor_SMD:R_0402_1005Metric -> Capacitor_SMD:C_0805_2012Metric_Pad1.18x1.45mm_HandSolder; Cost 0.0068 -> (none); Distributor LCSC -> (none); LCSC Part # C307454 -> (none); Manufacturer Samsung Electromechanics -> Samsung Microelectronics; Notes (none) -> 3.3V; P/N CL05X105KA5NQNC -> (none)
- C6: renamed from C102; footprint Resistor_SMD:R_0402_1005Metric -> Capacitor_SMD:C_0805_2012Metric_Pad1.18x1.45mm_HandSolder; Cost 0.0046 -> (none); Distributor LCSC -> (none); LCSC Part # C307331 -> (none); Manufacturer Samsung Electromechanics -> Samsung Microelectronics; Notes (none) -> 3.3V; P/N CL05B104KB54PNC -> (none)
- C7: renamed from C107; footprint (none) -> Capacitor_SMD:C_0805_2012Metric_Pad1.18x1.45mm_HandSolder; Manufacturer (none) -> Samsung Microelectronics; Notes (none) -> 3.3V
- C8: renamed from C118; footprint Resistor_SMD:R_0402_1005Metric -> Capacitor_SMD:C_0805_2012Metric_Pad1.18x1.45mm_HandSolder; Cost 0.0046 -> (none); Distributor LCSC -> (none); LCSC Part # C307331 -> (none); Manufacturer Samsung Electromechanics -> Samsung Microelectronics; Notes (none) -> 3.3V; P/N CL05B104KB54PNC -> (none)
- C9: renamed from C117; footprint Resistor_SMD:R_0402_1005Metric -> Capacitor_SMD:C_0805_2012Metric_Pad1.18x1.45mm_HandSolder; Cost 0.0068 -> (none); Distributor LCSC -> (none); LCSC Part # C307454 -> (none); Manufacturer Samsung Electromechanics -> Samsung Microelectronics; Notes (none) -> 3.3V; P/N CL05X105KA5NQNC -> (none)
- D1: renamed from D109; value 0.5 -> 0.35; footprint Diode_SMD:D_SMA -> Diode_SMD:D_SOD-123F; Cost 0.3 -> (none); Distributor Mouser -> (none); Manufacturer Vishay Electronics -> Diodes Incorporated; Notes 1.5A forward, 45Vrrm, sized to minimize turn off time (3.4.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 -> (none); P/N BYS10-45-E3/TR -> SBR3U40S1F-7
- D2: renamed from D108; footprint LED_SMD:LED_0402_1005Metric -> LED_SMD:LED_0805_2012Metric_Pad1.15x1.40mm_HandSolder; Cost 0.51 -> (none); Distributor Mouser -> (none); Manufacturer Wurth Elektronik -> (none); Notes Target V_FWD=3.1V, I_D=15mA, P_D=50mW -> (none); P/N 150040BS73220 -> (none)
- D3: renamed from D107; value 0.5 -> 0.35; footprint Diode_SMD:D_SMA -> Diode_SMD:D_SOD-123F; Cost 0.3 -> (none); Distributor Mouser -> (none); Manufacturer Vishay Electronics -> Diodes Incorporated; Notes 1.5A forward, 45Vrrm, sized to minimize turn off time (3.4.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 -> (none); P/N BYS10-45-E3/TR -> SBR3U40S1F-7
- D4: renamed from D101; value 0.5 -> 0.35; footprint Diode_SMD:D_SMA -> Diode_SMD:D_SOD-123F; Cost 0.3 -> (none); Distributor Mouser -> (none); Manufacturer Vishay Electronics -> Diodes Incorporated; Notes 1.5A forward, 45Vrrm, sized to minimize turn off time (3.4.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 -> (none); P/N BYS10-45-E3/TR -> SBR3U40S1F-7
- D5: renamed from D102; footprint LED_SMD:LED_0402_1005Metric -> LED_SMD:LED_0805_2012Metric_Pad1.15x1.40mm_HandSolder; Cost 0.51 -> (none); Distributor Mouser -> (none); Manufacturer Wurth Elektronik -> (none); Notes Target V_FWD=3.1V, I_D=15mA, P_D=50mW -> (none); P/N 150040BS73220 -> (none)
- D6: renamed from D103; value 0.5 -> 0.35; footprint Diode_SMD:D_SMA -> Diode_SMD:D_SOD-123F; Cost 0.3 -> (none); Distributor Mouser -> (none); Manufacturer Vishay Electronics -> Diodes Incorporated; Notes 1.5A forward, 45Vrrm, sized to minimize turn off time (3.4.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 -> (none); P/N BYS10-45-E3/TR -> SBR3U40S1F-7
- IC1: renamed from IC102; Distributor (none) -> Texas Instruments
- IC2: renamed from IC105; Distributor (none) -> Texas Instruments
- IC3: renamed from IC101; Distributor (none) -> Texas Instruments
- IC4: renamed from IC103; Distributor (none) -> Texas Instruments
- IC5: renamed from IC106; Distributor (none) -> Texas Instruments
- IC6: renamed from IC104; Distributor (none) -> Texas Instruments
- J5: renamed from J110; footprint (none) -> Connector_PinHeader_2.54mm:PinHeader_1x16_P2.54mm_Vertical
- Q1: renamed from Q110; value BSS127S -> Q_NMOS_GSD; footprint Package_TO_SOT_SMD:SOT-23 -> Package_TO_SOT_SMD:SOT-23-3; Cost 0.30 -> (none); Distributor Mouser -> (none); Manufacturer Diodes Incorporated -> Infineon; Notes 160O, 70mA, 1.25W -> (none); P/N BSS127S-7 -> BSS131
- Q6: renamed from Q104; value BSS127S -> Q_NMOS_GSD; footprint Package_TO_SOT_SMD:SOT-23 -> Package_TO_SOT_SMD:SOT-23-3; Cost 0.30 -> (none); Distributor Mouser -> (none); Manufacturer Diodes Incorporated -> Infineon; Notes 160O, 70mA, 1.25W -> (none); P/N BSS127S-7 -> BSS131
- R11: renamed from R109; footprint (none) -> Resistor_SMD:R_0805_2012Metric_Pad1.20x1.40mm_HandSolder; Manufacturer (none) -> Vishay / Dale
- R12: renamed from R126; footprint Resistor_SMD:R_0603_1608Metric -> Resistor_SMD:R_0805_2012Metric_Pad1.20x1.40mm_HandSolder; Cost 0.0009 -> (none); Distributor LCSC -> (none); LCSC Part # C22810 -> (none); Manufacturer Uniroyal -> Vishay / Dale; Notes Sized for 0.5A peak source current. -> 1A peak sink current.; P/N 0603WAF150JT5E -> (none)
- R13: renamed from R112; footprint (none) -> Resistor_SMD:R_0805_2012Metric_Pad1.20x1.40mm_HandSolder; Manufacturer (none) -> Vishay / Dale
- R14: renamed from R108; footprint Resistor_SMD:R_0603_1608Metric -> Resistor_SMD:R_0805_2012Metric_Pad1.20x1.40mm_HandSolder; Cost 0.0009 -> (none); Distributor LCSC -> (none); LCSC Part # C22810 -> (none); Manufacturer Uniroyal -> Vishay / Dale; Notes Sized for 0.5A peak source current. -> 0.5A peak source current.; P/N 0603WAF150JT5E -> (none)
- R15: renamed from R107; footprint (none) -> Resistor_SMD:R_0805_2012Metric_Pad1.20x1.40mm_HandSolder; Manufacturer (none) -> Vishay / Dale
- R16: renamed from R130; footprint (none) -> Resistor_SMD:R_0805_2012Metric_Pad1.20x1.40mm_HandSolder; Manufacturer (none) -> Vishay / Dale
- R17: renamed from R111; footprint (none) -> Resistor_SMD:R_0805_2012Metric_Pad1.20x1.40mm_HandSolder; Manufacturer (none) -> Vishay / Dale
- R18: renamed from R102; footprint Resistor_SMD:R_0603_1608Metric -> Resistor_SMD:R_0805_2012Metric_Pad1.20x1.40mm_HandSolder; Cost 0.0009 -> (none); Distributor LCSC -> (none); LCSC Part # C22810 -> (none); Manufacturer Uniroyal -> Vishay / Dale; Notes Sized for 0.5A peak source current. -> 0.5A peak source current.; P/N 0603WAF150JT5E -> (none)
- R19: renamed from R113; footprint (none) -> Resistor_SMD:R_0805_2012Metric_Pad1.20x1.40mm_HandSolder; Manufacturer (none) -> Vishay / Dale
- R2: renamed from R118; footprint (none) -> Resistor_SMD:R_0805_2012Metric_Pad1.20x1.40mm_HandSolder; Manufacturer (none) -> Vishay / Dale
- R20: renamed from R110; footprint (none) -> Resistor_SMD:R_0805_2012Metric_Pad1.20x1.40mm_HandSolder; Manufacturer (none) -> Vishay / Dale
- R21: renamed from R103; footprint Resistor_SMD:R_0603_1608Metric -> Resistor_SMD:R_0805_2012Metric_Pad1.20x1.40mm_HandSolder; Cost 0.0009 -> (none); Distributor LCSC -> (none); LCSC Part # C22810 -> (none); Manufacturer Uniroyal -> Vishay / Dale; Notes Sized for 0.5A peak source current. -> 1A peak sink current.; P/N 0603WAF150JT5E -> (none)
- R23: renamed from R123; footprint (none) -> Resistor_SMD:R_0805_2012Metric_Pad1.20x1.40mm_HandSolder; Manufacturer (none) -> Vishay / Dale
- R24: renamed from R105; footprint Resistor_SMD:R_0603_1608Metric -> Resistor_SMD:R_0805_2012Metric_Pad1.20x1.40mm_HandSolder; Cost 0.0009 -> (none); Distributor LCSC -> (none); LCSC Part # C22810 -> (none); Manufacturer Uniroyal -> Vishay / Dale; P/N 0603WAF150JT5E -> (none)
- R25: renamed from R106; footprint Resistor_SMD:R_0603_1608Metric -> Resistor_SMD:R_0805_2012Metric_Pad1.20x1.40mm_HandSolder; Cost 0.0009 -> (none); Distributor LCSC -> (none); LCSC Part # C22810 -> (none); Manufacturer Uniroyal -> Vishay / Dale; P/N 0603WAF150JT5E -> (none)
- R27: renamed from R122; footprint (none) -> Resistor_SMD:R_0805_2012Metric_Pad1.20x1.40mm_HandSolder; Manufacturer (none) -> Vishay / Dale
- R28: renamed from R124; value 150k -> 87.5k; footprint (none) -> Resistor_SMD:R_0805_2012Metric_Pad1.20x1.40mm_HandSolder; Manufacturer (none) -> Vishay / Dale
- R29: renamed from R125; footprint (none) -> Resistor_SMD:R_0805_2012Metric_Pad1.20x1.40mm_HandSolder; Manufacturer (none) -> Vishay / Dale
- R3: renamed from R119; footprint (none) -> Resistor_SMD:R_0805_2012Metric_Pad1.20x1.40mm_HandSolder; Manufacturer (none) -> Vishay / Dale
- R4: renamed from R129; footprint Resistor_SMD:R_0603_1608Metric -> Resistor_SMD:R_0805_2012Metric_Pad1.20x1.40mm_HandSolder; Cost 0.0009 -> (none); Distributor LCSC -> (none); LCSC Part # C22810 -> (none); Manufacturer Uniroyal -> Vishay / Dale; P/N 0603WAF150JT5E -> (none)
- R6: renamed from R128; footprint Resistor_SMD:R_0603_1608Metric -> Resistor_SMD:R_0805_2012Metric_Pad1.20x1.40mm_HandSolder; Cost 0.0009 -> (none); Distributor LCSC -> (none); LCSC Part # C22810 -> (none); Manufacturer Uniroyal -> Vishay / Dale; P/N 0603WAF150JT5E -> (none)
- R7: renamed from R120; footprint (none) -> Resistor_SMD:R_0805_2012Metric_Pad1.20x1.40mm_HandSolder; Manufacturer (none) -> Vishay / Dale
- R8: renamed from R114; footprint (none) -> Resistor_SMD:R_0805_2012Metric_Pad1.20x1.40mm_HandSolder; Manufacturer (none) -> Vishay / Dale
- R9: renamed from R101; footprint (none) -> Resistor_SMD:R_0805_2012Metric_Pad1.20x1.40mm_HandSolder; Manufacturer (none) -> Vishay / Dale
- U1: renamed from U104; Distributor (none) -> Texas Instruments
- U2: renamed from U101; Distributor (none) -> Texas Instruments
- renumbered J101 to J1, J103 to J2, J105 to J3, J107 to J4, J102 to J6, J104 to J7, J106 to J8, J108 to J9, TP104 to TP1, TP105 to TP2, TP106 to TP3, TP101 to TP4, TP102 to TP5, TP103 to TP6
Connections:
- net INA+: now also R1.1, R5.4; no longer R3.2
- net INB+: now also Q2.3 (D)
- net OUTA+: now also Q5.3 (D)
- net OUTB+: now also R26.1; no longer R27.2
- net at C4.2, U1.5 (VSSS): now also Q2.1 (S), Q3.1 (S)
- net at D2.1 (K): now also R10.1
- net at Q6.3 (D): now also R22.2
- net at Q1.3 (D): now also R10.2
- net at R7.2: now also R5.2
- net at R23.2: now also R26.3
- net at IC2.8 (VBUS), R2.1: now also R1.2
- net at C11.2, U2.5 (VSSS): now also Q4.1 (S), Q5.1 (S)
- net at D3.2 (A), R14.1: now also Q2.2 (G), Q3.2 (G)
- net at D4.2 (A), R18.1: now also Q4.2 (G), Q5.2 (G)
- net at D5.1 (K): now also R22.1
- new net: Q4.3 (D), R5.1
- new net: R3.2, R5.3
- new net: R26.2, R27.2
- new net: Q3.3 (D), R26.4
Other:
- moved on the sheet: D2, D5, R2, R23, R27, R28, R29, R3, R7
