File: hardware/mppt/power_converter.kicad_sch (KiCad schematic)
At the start: 31 parts, among them J301 Conn_01x01, J302 Conn_01x01, J303 CT3151, J304 CT3151, J305 CT3151, J306 CT3151, J307 Conn_01x01, J308 Conn_01x01

Commit message: remove testpoints, integrat 60% of layout
Parts:
- removed F301, F302: Fuse, footprints:littelfuse_65600001009, symbol Device:Fuse
- removed FC301, FC302: 65900000009, symbol littelfuse_021306_3MXP:65900000009
- removed FX301, FX302: 021306.3MXP, symbol littelfuse_021306_3MXP:021306_3MXP
- removed J303, J304, J305, J306: CT3151, footprints:caltest_ct3151, symbol caltest_ct3151:CT3151
- removed TP301, TP302, TP303: TestPoint, TestPoint:TestPoint_Keystone_5000-5004_Miniature, symbol Connector:TestPoint
- removed TP304, TP305, TP306, TP307, TP308, TP309, TP310, TP311, TP312, TP313, TP314, TP315, TP316, TP317: TestPoint_Small, TestPoint:TestPoint_Pad_D1.0mm, symbol Connector:TestPoint_Small
- renumbered J307 to J303, J308 to J304
Connections:
- net _IN+ is gone; now on net IN+: J301.1 (Pin_1)
