File: hardware/mppt/mppt.kicad_pcb (KiCad board)
At the start: 4 copper layers, 228.4 x 79.4 mm, 298 parts, among them IC1301 INA229AIDGSR, IC1501 LMR38010SDDAR, IC1502 TPS2121, IC5 APX803, IC801 INA229AIDGSR, IC901 SN74LVC08APWR, IC902 SN74LVC1G04DBVR, IC903 SN74HCS367PWR, IC904 SN74LVC2G32DCUR, J1501 Conn_01x02, J1502 CT3151, J1503 CT3151, J1504 CT3151, J303 CT3151, J304 CT3151, J305 CT3151, J306 CT3151, Q1 MMBT2222, Q1001 Q_NMOS_GDS, Q1101 Q_NMOS_SGD, Q1102 Q_NMOS_SGD, Q1201 Q_NMOS_SGD, Q1202 Q_NMOS_SGD, Q501 EPC2059, Q502 EPC2059, Q601 Q_NMOS_GDS, Q701 Q_NMOS_GDS, U1001 ADUM4221-1ARIZ, U1101 TPSI3050, U1201 TPSI3050, U1501 AP63205WU, U1502 TLV75733PDBV, U2 MIC5225-3.3, U3 74HC4050D

Commit message: remove testpoints, integrat 60% of layout
Parts:
- removed @HOLE0, @HOLE1, @HOLE2, @HOLE3, @HOLE4, @HOLE5, @HOLE6, @HOLE7, @HOLE8, @HOLE9: , 
- removed C1, C2: 10µF, Adafruit 1.14-inch 240x135 Color TFT:0805-NO
- removed C3: 0.1uF, Adafruit 1.14-inch 240x135 Color TFT:0805-NO
- removed CN1: , Adafruit 1.14-inch 240x135 Color TFT:MICROSD
- removed DISP1: DISP_LCD_GENERIC_SPI_1.14IN_240X135_WRAPUNDER, Adafruit 1.14-inch 240x135 Color TFT:TFT_1.14IN_240X135_WRAPUNDER
- removed F301, F302: Fuse, footprints:littelfuse_65600001009
- removed FID1, FID2: FIDUCIAL_1MM, Adafruit 1.14-inch 240x135 Color TFT:FIDUCIAL_1MM
- removed the H101 at (40.0, 30.0)
- removed the H101 at (172.9, 27.3)
- removed the H102 at (153.0, 30.0)
- removed the H102 at (212.8, 27.3)
- removed the H103 at (80.0, 95.0)
- removed the H103 at (184.9, 59.3)
- removed the H104 at (113.0, 95.0)
- removed the H104 at (200.9, 59.3)
- removed IC5: APX803, Adafruit 1.14-inch 240x135 Color TFT:SOT23
- removed J1502, J1503, J1504, J305, J306: CT3151, footprints:caltest_ct3151
- removed JP1: , Adafruit 1.14-inch 240x135 Color TFT:1X11_ROUND
- removed Q1: MMBT2222, Adafruit 1.14-inch 240x135 Color TFT:SOT23-WIDE
- removed R2, R8: 10K, Adafruit 1.14-inch 240x135 Color TFT:0603-NO
- removed R5: 22, Adafruit 1.14-inch 240x135 Color TFT:0603-NO
- removed R7: 1K, Adafruit 1.14-inch 240x135 Color TFT:0603-NO
- removed the REF** at (85.8, 74.6)
- removed the REF** at (120.6, 86.6)
- removed the REF** at (179.9, 27.3)
- removed the REF** at (201.9, 27.3)
- removed TP1001, TP1002, TP1003, TP1004, TP1005, TP1006, TP1007, TP1101, TP1102, TP1103, TP1104, TP1105, TP1201, TP1202, TP1203, TP1204, TP1205, TP1303, TP1304, TP1305, TP1306, TP1307, TP1509, TP1510, TP1511, TP1512, TP1513, TP1514, TP304, TP305, TP306, TP307, TP308, TP309, TP310, TP311, TP312, TP313, TP314, TP315, TP316, TP317, TP601, TP602, TP603, TP604, TP701, TP702, TP703, TP704, TP803, TP804, TP805, TP806, TP807: TestPoint_Small, TestPoint:TestPoint_Pad_D1.0mm
- removed TP1308, TP1309, TP808, TP809: TestPoint_2Pole, TestPoint:TestPoint_2Pads_Pitch2.54mm_Drill0.8mm
- removed TP1507, TP1508, TP301, TP302, TP303: TestPoint, TestPoint:TestPoint_Keystone_5000-5004_Miniature
- removed U$10, U$9: MOUNTINGHOLE2.5, Adafruit 1.14-inch 240x135 Color TFT:MOUNTINGHOLE_2.5_PLATED
- removed U$4: MICROSD, Adafruit 1.14-inch 240x135 Color TFT:ADAFRUIT_3.5MM
- removed U$6: , Adafruit 1.14-inch 240x135 Color TFT:PCBFEAT-REV-040
- removed U2: MIC5225-3.3, Adafruit 1.14-inch 240x135 Color TFT:SOT23-5
- removed U3: 74HC4050D, Adafruit 1.14-inch 240x135 Color TFT:SOIC16
- removed VR1001: PV36W104C01B00, footprints:bourns_PV36W201C01B00
- added C1401: 100n, Capacitor_SMD:C_0402_1005Metric_Pad0.74x0.62mm_HandSolder, B.Cu at (151.4, 73.3)
- added C1402: 100n, Capacitor_SMD:C_0402_1005Metric_Pad0.74x0.62mm_HandSolder, B.Cu at (157.5, 73.3)
- added C201: 10p, Capacitor_SMD:C_0402_1005Metric, B.Cu at (89.3, 62.8)
- added C202: 15p, Capacitor_SMD:C_0402_1005Metric, B.Cu at (82.5, 59.2)
- added C203: 100n, Capacitor_SMD:C_0402_1005Metric_Pad0.74x0.62mm_HandSolder, B.Cu at (87.6, 70.3)
- added C204: 10u, Capacitor_SMD:C_1206_3216Metric_Pad1.33x1.80mm_HandSolder, B.Cu at (103.0, 62.6)
- added C205: 100n, Capacitor_SMD:C_0402_1005Metric_Pad0.74x0.62mm_HandSolder, B.Cu at (98.7, 61.9)
- added C206: 10p, Capacitor_SMD:C_0402_1005Metric, B.Cu at (89.3, 65.0)
- added C207: 15p, Capacitor_SMD:C_0402_1005Metric, B.Cu at (85.7, 59.2)
- added C208: 100n, Capacitor_SMD:C_0402_1005Metric_Pad0.74x0.62mm_HandSolder, B.Cu at (106.0, 62.6)
- added C209: 100n, Capacitor_SMD:C_0402_1005Metric_Pad0.74x0.62mm_HandSolder, B.Cu at (98.7, 62.9)
- added C210: 4.7u, Capacitor_SMD:C_0603_1608Metric, B.Cu at (103.6, 69.3)
- added C211: 100n, Capacitor_SMD:C_0402_1005Metric_Pad0.74x0.62mm_HandSolder, B.Cu at (106.0, 69.2)
- added C212: 100n, Capacitor_SMD:C_0402_1005Metric_Pad0.74x0.62mm_HandSolder, B.Cu at (98.7, 69.8)
- added C213: 100n, Capacitor_SMD:C_0402_1005Metric_Pad0.74x0.62mm_HandSolder, B.Cu at (98.1, 66.7)
- added C214: 1u, Capacitor_SMD:C_0603_1608Metric_Pad1.08x0.95mm_HandSolder, B.Cu at (99.3, 66.1)
- added C401: 1u, Capacitor_SMD:C_0603_1608Metric_Pad1.08x0.95mm_HandSolder, B.Cu at (65.1, 70.0)
- added C402: 1u, Capacitor_SMD:C_0603_1608Metric_Pad1.08x0.95mm_HandSolder, B.Cu at (117.1, 92.1)
- added C403: 1u, Capacitor_SMD:C_0603_1608Metric_Pad1.08x0.95mm_HandSolder, B.Cu at (78.1, 57.1)
- added D201: RED, LED_SMD:LED_0805_2012Metric_Pad1.15x1.40mm_HandSolder, F.Cu at (109.9, 56.6)
- added D202: RED, LED_SMD:LED_0805_2012Metric_Pad1.15x1.40mm_HandSolder, F.Cu at (112.3, 56.6)
- added D203: RED, LED_SMD:LED_0805_2012Metric_Pad1.15x1.40mm_HandSolder, F.Cu at (114.8, 56.6)
- added FB201: FerriteBead, Resistor_SMD:R_0603_1608Metric_Pad0.98x0.95mm_HandSolder, B.Cu at (99.3, 68.6)
- added H101: MountingHole, MountingHole:MountingHole_2.7mm_M2.5_DIN965_Pad_TopBottom, F.Cu at (50.0, 50.0)
- added H102: MountingHole, MountingHole:MountingHole_2.7mm_M2.5_DIN965_Pad_TopBottom, F.Cu at (161.8, 50.0)
- added H103: MountingHole, MountingHole:MountingHole_2.7mm_M2.5_DIN965_Pad_TopBottom, F.Cu at (77.0, 126.0)
- added H104: MountingHole, MountingHole:MountingHole_2.7mm_M2.5_DIN965_Pad_TopBottom, F.Cu at (111.5, 126.0)
- added H1401: MountingHole, MountingHole:MountingHole_2.7mm_M2.5_DIN965_Pad_TopBottom, F.Cu at (119.8, 72.8)
- added H1402: MountingHole, MountingHole:MountingHole_2.7mm_M2.5_DIN965_Pad_TopBottom, F.Cu at (146.4, 72.7)
- added J1401: Conn_01x04, Connector_Molex:Molex_Micro-Fit_3.0_43650-0415_1x04_P3.00mm_Vertical, F.Cu at (162.3, 70.1)
- added J1402: Conn_01x02, Connector_PinHeader_2.54mm:PinHeader_1x02_P2.54mm_Vertical, F.Cu at (153.2, 80.8)
- added J1403: Conn_02x04_Odd_Even, Connector_PinHeader_2.54mm:PinHeader_2x04_P2.54mm_Vertical, F.Cu at (112.9, 49.8)
- added J1404: Conn_01x11, Connector_PinHeader_2.54mm:PinHeader_1x11_P2.54mm_Vertical, F.Cu at (120.4, 50.0)
- added J1405: USB_C_Plug_USB2.0, Connector_USB:USB_C_Receptacle_GCT_USB4105-xx-A_16P_TopMnt_Horizontal, F.Cu at (162.8, 58.9)
- added J301: Conn_01x01, footprints:ke_7771_SEMS, F.Cu at (49.9, 119.5)
- added J302: Conn_01x01, footprints:ke_7771_SEMS, F.Cu at (65.0, 119.5)
- added J401: Conn_01x04, Connector_Molex:Molex_Micro-Fit_3.0_43650-0415_1x04_P3.00mm_Vertical, F.Cu at (93.2, 51.9)
- added J402: Conn_01x03, Connector_Molex:Molex_Micro-Fit_3.0_43650-0315_1x03_P3.00mm_Vertical, F.Cu at (75.4, 51.9)
- added JP201: Jumper_3_Bridged12, Connector_PinSocket_2.54mm:PinSocket_1x03_P2.54mm_Vertical, F.Cu at (94.5, 58.7)
- added NT1401: NetTie_2, NetTie:NetTie-2_SMD_Pad2.0mm, B.Cu at (154.1, 71.2)
- added R1007: R_DT, Resistor_SMD:R_0805_2012Metric_Pad1.20x1.40mm_HandSolder, F.Cu at (237.4, 118.6)
- added R1401: 120, Resistor_SMD:R_0603_1608Metric_Pad0.98x0.95mm_HandSolder, B.Cu at (154.3, 77.6)
- added R1402: 100k, Resistor_SMD:R_0603_1608Metric_Pad0.98x0.95mm_HandSolder, B.Cu at (102.4, 54.2)
- added R1403: 100k, Resistor_SMD:R_0603_1608Metric_Pad0.98x0.95mm_HandSolder, B.Cu at (106.5, 56.2)
- added R1404: 100k, Resistor_SMD:R_0603_1608Metric_Pad0.98x0.95mm_HandSolder, B.Cu at (102.4, 56.2)
- added R1405: 5.1k, Resistor_SMD:R_0603_1608Metric_Pad0.98x0.95mm_HandSolder, F.Cu at (154.4, 56.0)
- added R1406: 5.1k, Resistor_SMD:R_0603_1608Metric_Pad0.98x0.95mm_HandSolder, F.Cu at (154.4, 61.8)
- added R201: 3.3k, Resistor_SMD:R_0603_1608Metric_Pad0.98x0.95mm_HandSolder, B.Cu at (109.9, 56.6)
- added R202: 3.3k, Resistor_SMD:R_0603_1608Metric_Pad0.98x0.95mm_HandSolder, B.Cu at (112.3, 56.6)
- added R203: 0, Resistor_SMD:R_0805_2012Metric_Pad1.20x1.40mm_HandSolder, B.Cu at (92.8, 63.5)
- added R204: 100k, Resistor_SMD:R_0603_1608Metric_Pad0.98x0.95mm_HandSolder, B.Cu at (92.8, 56.6)
- added R205: 3.3k, Resistor_SMD:R_0603_1608Metric_Pad0.98x0.95mm_HandSolder, B.Cu at (114.8, 56.6)
- added R401: 205, Resistor_SMD:R_0603_1608Metric_Pad0.98x0.95mm_HandSolder, B.Cu at (66.9, 70.0)
- added R402: 205, Resistor_SMD:R_0603_1608Metric_Pad0.98x0.95mm_HandSolder, B.Cu at (119.0, 92.1)
- added R403: 205, Resistor_SMD:R_0603_1608Metric_Pad0.98x0.95mm_HandSolder, B.Cu at (78.1, 52.8)
- added REF**: OSHW-Logo2_9.8x8mm_Copper, Symbol:OSHW-Logo2_9.8x8mm_Copper, B.Cu at (102.8, 126.0)
- added SW201: SW_SPST, Button_Switch_THT:SW_PUSH_6mm, F.Cu at (91.5, 72.5)
- added TP201: TestPoint_Small, TestPoint:TestPoint_Pad_D1.0mm, B.Cu at (104.5, 65.9)
- added TP202: TestPoint_Small, TestPoint:TestPoint_Pad_D1.0mm, B.Cu at (102.0, 65.9)
- added TP203: TestPoint_Small, TestPoint:TestPoint_Pad_D1.0mm, F.Cu at (99.0, 49.2)
- added TP204: TestPoint_Small, TestPoint:TestPoint_Pad_D1.0mm, F.Cu at (99.0, 51.7)
- added TP205: TestPoint_Small, TestPoint:TestPoint_Pad_D1.0mm, F.Cu at (114.2, 67.8)
- added TP206: TestPoint_Small, TestPoint:TestPoint_Pad_D1.0mm, F.Cu at (116.1, 66.5)
- added TP207: TestPoint_Small, TestPoint:TestPoint_Pad_D1.0mm, F.Cu at (114.2, 65.2)
- added TP208: TestPoint_Small, TestPoint:TestPoint_Pad_D1.0mm, F.Cu at (112.4, 66.5)
- added TP209: TestPoint_Small, TestPoint:TestPoint_Pad_D1.0mm, F.Cu at (116.1, 64.0)
- added TP210: TestPoint_Small, TestPoint:TestPoint_Pad_D1.0mm, F.Cu at (112.4, 64.0)
- added U1401: ISO1044BD, Package_SO:SOIC-8_3.9x4.9mm_P1.27mm, F.Cu at (153.9, 75.2)
- added U1402: USBLC6-2SC6, Package_TO_SOT_SMD:SOT-23-6, F.Cu at (154.0, 58.9)
- added U201: STM32F446RETx, Package_QFP:LQFP-64_10x10mm_P0.5mm, F.Cu at (102.0, 65.9)
- added U401: MCP9700Ax-ELT, Package_TO_SOT_SMD:SOT-353_SC-70-5, F.Cu at (66.0, 70.0)
- added U402: MCP9700Ax-ELT, Package_TO_SOT_SMD:SOT-353_SC-70-5, F.Cu at (118.0, 92.1)
- added Y201: 16MHz, Crystal:Crystal_SMD_Abracon_ABM8G-4Pin_3.2x2.5mm, F.Cu at (89.3, 63.9)
- added Y202: 32kHz, Crystal:Crystal_SMD_Abracon_ABS25-4Pin_8.0x3.8mm, F.Cu at (84.1, 61.4)
- C1104, C1201, C1202, C1204, D701, D702, Q701, R1201: moved to B.Cu
- C1302, C1501, C1504, C802, D1101, D1201, R703, U1101, U1201: moved to F.Cu
- C1502, C1503, C503, C506: footprint Capacitor_SMD:C_2220_5750Metric_Pad1.97x5.40mm_HandSolder -> Capacitor_SMD:C_2220_5750Metric
- C1505: footprint Capacitor_SMD:C_1206_3216Metric_Pad1.33x1.80mm_HandSolder -> Capacitor_SMD:C_0805_2012Metric; moved to B.Cu
- C1508, C1514, C1515: footprint Capacitor_SMD:C_1210_3225Metric_Pad1.33x2.70mm_HandSolder -> Capacitor_SMD:C_1206_3216Metric
- C1509: footprint Capacitor_SMD:C_1210_3225Metric_Pad1.33x2.70mm_HandSolder -> Capacitor_SMD:C_1206_3216Metric; moved to B.Cu
- C501, C505: footprint Capacitor_SMD:C_1206_3216Metric_Pad1.33x1.80mm_HandSolder -> Capacitor_SMD:C_0805_2012Metric
- C502, C507: footprint Capacitor_SMD:C_2220_5750Metric_Pad1.97x5.40mm_HandSolder -> Capacitor_SMD:C_2220_5750Metric; moved to B.Cu
- J303, J304: value CT3151 -> Conn_01x01; footprint footprints:caltest_ct3151 -> footprints:ke_7771_SEMS
- R1102, R1103, R1202, R1203: footprint Resistor_SMD:R_1210_3225Metric_Pad1.30x2.65mm_HandSolder -> Resistor_SMD:R_0603_1608Metric; moved to B.Cu
- R1303, R1305, R803, R805: footprint Resistor_SMD:R_0603_1608Metric_Pad0.98x0.95mm_HandSolder -> Resistor_SMD:R_0603_1608Metric
- R601, R602: footprint Resistor_SMD:R_1210_3225Metric_Pad1.30x2.65mm_HandSolder -> Resistor_SMD:R_0603_1608Metric
- R701, R702: footprint Resistor_SMD:R_1210_3225Metric_Pad1.30x2.65mm_HandSolder -> Resistor_SMD:R_0603_1608Metric; moved to F.Cu
- TP1301, TP1302, TP801, TP802: value TestPoint_Small -> TestPoint_2Pole; footprint TestPoint:TestPoint_Pad_D1.0mm -> TestPoint:TestPoint_2Pads_Pitch2.54mm_Drill0.8mm
- TP1501, TP1502, TP1503, TP1504, TP1505, TP1506: value TestPoint -> TestPoint_Small; footprint TestPoint:TestPoint_Keystone_5000-5004_Miniature -> TestPoint:TestPoint_Pad_D1.0mm
- moved TP1501 167.2 mm to (49.0, 78.9), turned to 0 degrees
- moved IC1501 166.8 mm to (50.1, 98.0)
- moved R1501 166.8 mm to (54.1, 101.9)
- moved R1502 166.8 mm to (54.1, 100.0)
- moved R1507 166.8 mm to (52.1, 100.0)
- moved R1516 166.7 mm to (54.1, 95.8)
- moved C1505 166.7 mm to (49.9, 103.2)
- moved C1506 166.4 mm to (48.9, 93.3)
- moved NT1501 166.1 mm to (51.0, 106.0), turned to 0 degrees
- moved C1502 166.1 mm to (51.0, 105.1)
- moved C1503 166.1 mm to (51.0, 105.1)
- moved R1513 165.5 mm to (52.1, 92.1)
- moved R1514 165.5 mm to (54.1, 92.1)
- moved R1515 165.5 mm to (54.1, 93.9)
- moved L1501 156.7 mm to (50.9, 86.2), turned to 0 degrees
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Connections:
- net /power_converter/Load Switch Sink/I+ renamed /power_converter/Load Switch Source/I+
- net /power_converter/Load Switch Source/I- renamed /power_converter/Load Switch Sink/I-
- C1103 pad 1: /power_converter/Load Switch Source/VDDH -> /power_converter/Load Switch Sink/VDDH
- C1104 pad 2: /power_converter/Load Switch Source/VSSS -> /power_converter/Load Switch Sink/VSSS
- C1203 pad 1: /power_converter/Load Switch Sink/VDDH -> /power_converter/Load Switch Source/VDDH
- C1204 pad 2: /power_converter/Load Switch Sink/VSSS -> /power_converter/Load Switch Source/VSSS
- C1501 pad 1: (no net) -> +12L
- C1502 pad 2: /VI- -> GND
- C1503 pad 2: /VI- -> GND
- C1504 pad 1: (no net) -> +12C
- C1505 pad 2: /VI- -> GND
- C1506 pad 1: (no net) -> Net-(IC1501-SW)
- C1506 pad 2: (no net) -> Net-(IC1501-BOOT)
- C1507 pad 1: (no net) -> Net-(IC1502-SS)
- C1508 pad 1: (no net) -> +12V
- C1509 pad 1: (no net) -> +12C
- C1510 pad 1: (no net) -> +12V
- C1513 pad 1: (no net) -> Net-(U1501-BST)
- C1513 pad 2: (no net) -> Net-(U1501-SW)
- D1501 pad 2: (no net) -> +12L
- D1502 pad 2: (no net) -> +12C
- D1503 pad 2: (no net) -> Net-(D1503-A)
- D1505 pad 2: (no net) -> Net-(D1505-A)
- D1506 pad 2: (no net) -> Net-(D1506-A)
- IC1501 pad 2: (no net) -> Net-(IC1501-EN)
- IC1501 pad 4: (no net) -> Net-(IC1501-RT/SYNC)
- IC1501 pad 5: (no net) -> /power regulation/BUCK_FB
- IC1501 pad 6: (no net) -> /power regulation/BUCK_PG
- IC1501 pad 7: (no net) -> Net-(IC1501-BOOT)
- IC1501 pad 8: (no net) -> Net-(IC1501-SW)
- IC1502 pad 1: (no net) -> +12V
- IC1502 pad 10: (no net) -> Net-(IC1502-ILIM)
- IC1502 pad 11: (no net) -> Net-(IC1502-SS)
- IC1502 pad 2: (no net) -> +12C
- IC1502 pad 3: (no net) -> /power regulation/CP2
- IC1502 pad 4: (no net) -> /power regulation/OV2
- IC1502 pad 5: (no net) -> /power regulation/OV1
- IC1502 pad 6: (no net) -> /power regulation/PR1
- IC1502 pad 7: (no net) -> +12L
- IC1502 pad 8: (no net) -> +12V
- J1501 pad 1: (no net) -> +12L
- J303 pad 1: /power_converter/_IN+ -> /power_converter/OUT+
- J304 pad 1: /VI- -> /power_converter/OUT-
- JP1501 pad 1: (no net) -> Net-(JP1501-A)
- JP1501 pad 3: (no net) -> /VUSB
- L1501 pad 1: (no net) -> Net-(IC1501-SW)
- L1501 pad 2: (no net) -> +12C
- L1502 pad 1: (no net) -> Net-(U1501-SW)
- L1502 pad 2: (no net) -> Net-(JP1501-A)
- Q1101 pad 1: /power_converter/Load Switch Source/VSSS -> /power_converter/Load Switch Sink/VSSS
- Q1102 pad 1: /power_converter/Load Switch Source/VSSS -> /power_converter/Load Switch Sink/VSSS
- Q1201 pad 1: /power_converter/Load Switch Sink/VSSS -> /power_converter/Load Switch Source/VSSS
- Q1202 pad 1: /power_converter/Load Switch Sink/VSSS -> /power_converter/Load Switch Source/VSSS
- R1102 pad 2: /power_converter/Load Switch Source/VDRV -> /power_converter/Load Switch Sink/VDRV
- R1103 pad 2: /power_converter/Load Switch Source/VDRV -> /power_converter/Load Switch Sink/VDRV
- R1202 pad 2: /power_converter/Load Switch Sink/VDRV -> /power_converter/Load Switch Source/VDRV
- R1203 pad 2: /power_converter/Load Switch Sink/VDRV -> /power_converter/Load Switch Source/VDRV
- R1304 pad 4: /power_converter/Power Monitor Sink/I- -> /power_converter/OUT+
- R1501 pad 2: (no net) -> Net-(IC1501-EN)
- R1502 pad 1: (no net) -> Net-(IC1501-EN)
- R1503 pad 1: (no net) -> +12L
- R1503 pad 2: (no net) -> /power regulation/OV1
- R1504 pad 1: (no net) -> /power regulation/OV1
- R1505 pad 1: (no net) -> +12C
- R1505 pad 2: (no net) -> /power regulation/OV2
- R1506 pad 1: (no net) -> /power regulation/OV2
- R1507 pad 1: (no net) -> Net-(IC1501-RT/SYNC)
- R1508 pad 1: (no net) -> +12L
- R1508 pad 2: (no net) -> /power regulation/PR1
- R1509 pad 1: (no net) -> /power regulation/PR1
- R1510 pad 1: (no net) -> +12C
- R1510 pad 2: (no net) -> /power regulation/CP2
- R1511 pad 1: (no net) -> /power regulation/CP2
- R1512 pad 1: (no net) -> Net-(IC1502-ILIM)
- R1513 pad 1: (no net) -> +12C
- R1513 pad 2: (no net) -> /power regulation/BUCK_PG
- R1514 pad 1: (no net) -> +12C
- R1514 pad 2: (no net) -> Net-(R1514-Pad2)
- R1515 pad 1: (no net) -> Net-(R1514-Pad2)
- R1515 pad 2: (no net) -> /power regulation/BUCK_FB
- R1516 pad 1: (no net) -> /power regulation/BUCK_FB
- R1517 pad 1: (no net) -> +12V
- R1517 pad 2: (no net) -> Net-(D1503-A)
- R1518 pad 2: (no net) -> Net-(D1505-A)
- R1519 pad 2: (no net) -> Net-(D1506-A)
- TP1301 pad 1: /MON_SPI_CLK -> /power_converter/Power Monitor Sink/VBUS
- TP1302 pad 1: /MON_SPI_CIPO -> /power_converter/Power Monitor Sink/IN+
- TP1501 pad 1: /VI+ -> +12C
- TP1502 pad 1: /VI- -> GND
- TP1503 pad 1: (no net) -> +12L
- TP1504 pad 1: GND -> +12V
- TP1505 pad 1: (no net) -> +5V
- TP1506 pad 1: (no net) -> +3V3
- TP801 pad 1: /MON_SPI_CLK -> /power_converter/Power Monitor Source/VBUS
- TP802 pad 1: /MON_SPI_CIPO -> /power_converter/Power Monitor Source/IN+
- U1101 pad 5: /power_converter/Load Switch Source/VSSS -> /power_converter/Load Switch Sink/VSSS
- U1101 pad 7: /power_converter/Load Switch Source/VDDH -> /power_converter/Load Switch Sink/VDDH
- U1101 pad 8: /power_converter/Load Switch Source/VDRV -> /power_converter/Load Switch Sink/VDRV
- U1201 pad 5: /power_converter/Load Switch Sink/VSSS -> /power_converter/Load Switch Source/VSSS
- U1201 pad 7: /power_converter/Load Switch Sink/VDDH -> /power_converter/Load Switch Source/VDDH
- U1201 pad 8: /power_converter/Load Switch Sink/VDRV -> /power_converter/Load Switch Source/VDRV
- U1501 pad 1: (no net) -> Net-(JP1501-A)
- U1501 pad 2: (no net) -> +12V
- U1501 pad 3: (no net) -> +12V
- U1501 pad 5: (no net) -> Net-(U1501-SW)
- U1501 pad 6: (no net) -> Net-(U1501-BST)
- U1502 pad 4: (no net) -> unconnected-(U1502-NC-Pad4)
Routing:
- net (no net): track 582.7 -> 0.00 mm, vias 58 -> 0
- net /power_converter/~{MON_ALERT}: track 166.5 -> 25.0 mm, vias 11 -> 3
- net /MON_SPI_CLK: track 134.4 -> 0.00 mm, vias 4 -> 0
- net /VUSB: track 0.00 -> 131.5 mm, vias 0 -> 8
- net /MON_SPI_COPI: track 131.5 -> 0.00 mm, vias 4 -> 0
- net /MON_SPI_CIPO: track 128.6 -> 0.00 mm, vias 2 -> 0
- net /MON_IN_CS: track 67.0 -> 0.00 mm, vias 3 -> 0
- net /MON_OUT_CS: track 65.2 -> 0.00 mm, vias 1 -> 0
- net +5V: track 126.3 -> 184.9 mm, vias 9 -> 18
- net /VI-: track 60.6 -> 11.7 mm, vias 89 -> 0
- net /SDC_CS: track 0.00 -> 47.9 mm, vias 0 -> 2
- net /USB-: track 0.00 -> 47.7 mm
- net /CAN_TX: track 0.00 -> 47.1 mm
- net /USB+: track 0.00 -> 46.9 mm
- net /CAN_RX: track 0.00 -> 46.7 mm
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- added copper zone on F.Cu, net +12V
- added copper zone on B.Cu, net +3V3
- added copper zone on In1.Cu, net +3V3
- added copper zone on In2.Cu, net +3V3
- added copper zone on B.Cu, net +5V
- added copper zone on In1.Cu, net +5V
- added copper zone on B.Cu, net /VUSB
- added copper zone on B.Cu, net GND1
- removed copper zone on F.Cu, net (none)
- removed copper zone on B.Cu, net /VI+
- removed copper zone on F.Cu, net /VI+
- removed copper zone on In1.Cu, net /VI+
- removed copper zone on In2.Cu, net /VI+
- removed copper zone on B.Cu, net /VI-
- removed copper zone on F.Cu, net /VI-
- removed copper zone on In1.Cu, net /VI-
- removed copper zone on In2.Cu, net /VI-
- removed copper zone on B.Cu, net /power_converter/Active Load Sink/V+
- removed copper zone on F.Cu, net /power_converter/Active Load Sink/V+
- removed copper zone on In1.Cu, net /power_converter/Active Load Sink/V+
- removed copper zone on In2.Cu, net /power_converter/Active Load Sink/V+
- removed copper zone on B.Cu, net /power_converter/Active Load Source/V+
- removed copper zone on F.Cu, net /power_converter/Active Load Source/V+
- removed copper zone on In1.Cu, net /power_converter/Active Load Source/V+
- removed copper zone on In2.Cu, net /power_converter/Active Load Source/V+
- removed copper zone on F.Cu, net /power_converter/Load Switch Sink/I-
- removed copper zone on In1.Cu, net /power_converter/Load Switch Sink/I-
- removed copper zone on F.Cu, net /power_converter/Load Switch Source/I+
- removed copper zone on In1.Cu, net /power_converter/Load Switch Source/I+
- removed copper zone on B.Cu, net /power_converter/OUT+
- removed copper zone on F.Cu, net /power_converter/OUT+
- removed copper zone on In1.Cu, net /power_converter/OUT+
- removed copper zone on In2.Cu, net /power_converter/OUT+
- removed copper zone on B.Cu, net /power_converter/OUT-
- removed copper zone on F.Cu, net /power_converter/OUT-
- removed copper zone on In1.Cu, net /power_converter/OUT-
- removed copper zone on In2.Cu, net /power_converter/OUT-
- removed copper zone on B.Cu, net /power_converter/Power Monitor Sink/I-
- removed copper zone on F.Cu, net /power_converter/Power Monitor Sink/I-
- removed copper zone on In1.Cu, net /power_converter/Power Monitor Sink/I-
- removed copper zone on In2.Cu, net /power_converter/Power Monitor Sink/I-
- removed copper zone on B.Cu, net /power_converter/_IN+
- removed copper zone on F.Cu, net /power_converter/_IN+
- removed copper zone on In1.Cu, net /power_converter/_IN+
- removed copper zone on In2.Cu, net /power_converter/_IN+
- removed copper zone on B.Cu, net GND
- removed copper zone on F.Cu, net GND
- removed copper zone on In1.Cu, net GND
- removed copper zone on In2.Cu, net GND
Other:
- board size 228.4 x 79.4 mm -> 121.5 x 85 mm
- board text added: "M2"
- board text added: "M2.5"
- board text added: "Mighty MPPT v0.1.0rc"
- board text added: "Swap down to 0603."
- board text removed: "0-80V"
- board text removed: "12C"
- board text removed: "12L"
- board text removed: "3V"
- board text removed: "DC"
- board text removed: "GND"
- board text removed: "LIT"
- board text removed: "MISO"
- board text removed: "MOSI"
- board text removed: "Mighty MPPT Power Path v0.1.0rc M.Y. & J.P."
- board text removed: "Mighty MPPT Power Regulation Breakout v0.1.0rc Matthew Yu & Jacob Pustilnik"
- board text removed: "RST"
- board text removed: "SCK"
- board text removed: "SDCS"
- board text removed: "ST7789 1.14""
- board text removed: "TFTCS"
- board text removed: "VI+"
- board text removed: "VI-"
- board text removed: "Vin"
- board text removed: "Vin/Vlogic:3-5VDC"
- board text removed: "adafruit 240x135 Color TFT"

Commit message: swap can net tie to solder bridge for iso, 80% done layout
Parts:
- removed NT1401: NetTie_2, NetTie:NetTie-2_SMD_Pad2.0mm
- added JP1401: SolderJumper_2_Open, Jumper:SolderJumper-2_P1.3mm_Open_TrianglePad1.0x1.5mm, F.Cu at (154.8, 70.7)
- added JP1402: SolderJumper_2_Open, Jumper:SolderJumper-2_P1.3mm_Open_TrianglePad1.0x1.5mm, F.Cu at (154.8, 67.5)
- NT1001, NT1301: moved to F.Cu
- moved C1002 128.0 mm to (129.0, 78.2)
- moved C1003 128.0 mm to (131.6, 86.7)
- moved C1004 128.0 mm to (123.9, 86.7)
- moved C1005 128.0 mm to (131.6, 88.8)
- moved C1006 128.0 mm to (125.3, 88.8)
- moved D1004 128.0 mm to (125.2, 83.3)
- moved R1006 128.0 mm to (131.7, 83.5)
- moved U1001 128.0 mm to (127.8, 83.5)
- moved Q1001 126.0 mm to (126.3, 72.7)
- moved R1001 126.0 mm to (126.3, 76.9)
- moved C1001 126.0 mm to (131.6, 74.6)
- moved R1007 124.4 mm to (119.4, 79.4)
- moved NT1001 87.1 mm to (111.9, 80.9), turned to 0 degrees
- moved TP506 51.1 mm to (135.6, 94.4)
- moved TP504 45.8 mm to (133.1, 98.0), turned to 0 degrees
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Connections:
- C1402 pad 1: +5V -> /communication_interfaces/VCAN
- J1401 pad 1: +5V -> /communication_interfaces/VCAN
- U1401 pad 8: +5V -> /communication_interfaces/VCAN
Routing:
- net +3V3: track 276.8 -> 350.7 mm, vias 36 -> 41
- net +5V: track 184.9 -> 244.4 mm, vias 18 -> 22
- net /TEMP_BOARD: track 6.01 -> 33.7 mm
- net GND: track 107.4 -> 134.1 mm, vias 65 -> 70
- net /power_converter/OUT-: track 44.8 -> 18.6 mm, vias 11 -> 55
- net /power_converter/Active Load Sink/V+: track 3.06 -> 22.7 mm, vias 6 -> 24
- net /VI-: track 11.7 -> 29.8 mm, vias 0 -> 169
- net /VUSB: track 131.5 -> 118.0 mm, vias 8 -> 13
- net /power_converter/Gate Driver/CONV_PWM: track 17.1 -> 4.08 mm
- net /VI+: track 0.47 -> 13.1 mm, vias 1 -> 15
- net /communication_interfaces/CAN+: track 2.37 -> 14.6 mm, vias 1 -> 0
- net /communication_interfaces/CAN-: track 3.84 -> 14.9 mm
- net /power_converter/Load Switch Source/VSSS: track 12.3 -> 23.2 mm, vias 1 -> 6
- net GNDPWR: track 26.2 -> 15.4 mm
- net Net-(D602-K): track 11.8 -> 2.30 mm
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- added copper zone on F.Cu, net +12C
- added copper zone on F.Cu, net +12L
- added copper zone on B.Cu, net /VI+
- added copper zone on F.Cu, net /VI+
- added copper zone on In1.Cu, net /VI+
- added copper zone on In2.Cu, net /VI+
- added copper zone on B.Cu, net /VI-
- added copper zone on F.Cu, net /VI-
- added copper zone on In1.Cu, net /VI-
- added copper zone on In2.Cu, net /VI-
- added copper zone on F.Cu, net /VUSB
- added copper zone on In1.Cu, net /VUSB
- added copper zone on In2.Cu, net /VUSB
- added copper zone on F.Cu, net /communication_interfaces/VCAN
- added copper zone on B.Cu, net /power_converter/Active Load Sink/V+
- added copper zone on In2.Cu, net /power_converter/Active Load Sink/V+
- added copper zone on B.Cu, net /power_converter/Active Load Source/V+
- added copper zone on F.Cu, net /power_converter/Load Switch Sink/I-
- added copper zone on F.Cu, net /power_converter/Load Switch Source/I+
- added copper zone on B.Cu, net /power_converter/Load Switch Source/VSSS
- added copper zone on F.Cu, net /power_converter/Load Switch Source/VSSS
- added copper zone on In1.Cu, net /power_converter/Load Switch Source/VSSS
- added copper zone on In2.Cu, net /power_converter/Load Switch Source/VSSS
- added copper zone on B.Cu, net /power_converter/OUT+
- added copper zone on F.Cu, net /power_converter/OUT+
- added copper zone on In1.Cu, net /power_converter/OUT+
- added copper zone on In2.Cu, net /power_converter/OUT+
- added copper zone on B.Cu, net /power_converter/OUT-
- added copper zone on F.Cu, net /power_converter/OUT-
- added copper zone on In1.Cu, net /power_converter/OUT-
- added copper zone on In2.Cu, net /power_converter/OUT-
- added copper zone on B.Cu, net GND
- added copper zone on F.Cu, net GND
- added copper zone on In1.Cu, net GND
- added copper zone on In2.Cu, net GND
- added copper zone on In1.Cu, net GND1
- added copper zone on In2.Cu, net GND1
- removed copper zone on B.Cu, net /VUSB
